Commit message: Update robot code

File: urdf/gazebo_control.xacro (robot description, xacro)
@@ -1,27 +1,20 @@
 <?xml version="1.0"?>
 <robot xmlns:xacro="http://www.ros.org/wiki/xacro">
-    <gazebo>
-        <plugin name="skid_steer_drive_controller" filename="libgazebo_ros_skid_steer_drive.so">
-            <updateRate>100.0</updateRate>
-            <robotNamespace>/</robotNamespace>
-            <leftFrontJoint>front_left_wheel_joint</leftFrontJoint>
-            <rightFrontJoint>front_right_wheel_joint</rightFrontJoint>
-            <leftRearJoint>rear_left_wheel_joint</leftRearJoint>
-            <rightRearJoint>rear_right_wheel_joint</rightRearJoint>
-            <wheelSeparation>0.35</wheelSeparation>
-            <wheelDiameter>0.1</wheelDiameter>
-            <torque>20</torque>
-            <commandTopic>cmd_vel</commandTopic>
-            <odometryTopic>odom</odometryTopic>
-            <odometryFrame>odom</odometryFrame>
-            <robotBaseFrame>base_link</robotBaseFrame>
-            <broadcastTF>true</broadcastTF>
-        </plugin>
-        <plugin name="joint_state_publisher" filename="libgazebo_ros_joint_state_publisher.so">
-            <robotNamespace>/</robotNamespace>
-            <jointName>front_left_wheel_joint, front_right_wheel_joint, rear_left_wheel_joint, rear_right_wheel_joint</jointName>
-            <updateRate>50.0</updateRate>
-            <alwaysOn>true</alwaysOn>
-        </plugin>
-    </gazebo>
+  <gazebo>
+    <plugin name="mecanum_controller" filename="libgazebo_ros_planar_move.so">
+      <commandTopic>cmd_vel</commandTopic>
+      <odometryTopic>odom</odometryTopic>
+      <odometryFrame>odom</odometryFrame>
+      <odometryRate>20.0</odometryRate>
+      <robotBaseFrame>base_link</robotBaseFrame>
+      <accelX>10.0</accelX>
+      <accelY>10.0</accelY>
+      <accelTheta>20.0</accelTheta>
+    </plugin> <plugin name="joint_state_publisher" filename="libgazebo_ros_joint_state_publisher.so">
+      <robotNamespace>/</robotNamespace>
+      <jointName>front_left_wheel_joint, front_right_wheel_joint, rear_left_wheel_joint, rear_right_wheel_joint</jointName>
+      <updateRate>50.0</updateRate>
+      <alwaysOn>true</alwaysOn>
+    </plugin>
+  </gazebo>
 </robot>

File: urdf/robot_core.xacro (robot description, xacro)
@@ -1,104 +1,69 @@
 <?xml version="1.0"?>
-<robot xmlns:xacro="http://www.ros.org/wiki/xacro" name="mobile_robot">
-  <link name="base_link">
-  </link>
-  <xacro:property name="height" value="0.4" />
-  <xacro:property name="width" value="0.4" />
-  <xacro:property name="depth" value="0.1" />
-  <link name="chassis">
-    <visual>
-      <geometry>
-        <box size="${height} ${width} ${depth}"/>
-      </geometry>
-    </visual>
-    <collision>
-      <geometry>
-        <box size="${height} ${width} ${depth}"/>
-      </geometry>
-    </collision>
-    <inertial>
-      <mass value="5.0"/> <inertia ixx="0.1" ixy="0.0" ixz="0.0" iyy="0.1" iyz="0.0" izz="0.1"/>
-    </inertial>
-  </link>
-  <gazebo reference="chassis">
-    <material>Gazebo/Red</material>
-  </gazebo>
-  <joint name="chassis_joint" type="fixed">
-    <parent link="base_link"/>
-    <child link="chassis"/>
-  </joint>
-  <material name="blue">
-    <color rgba="0 0 0.8 1"/>
-  </material>
-  <xacro:property name="wheel_height" value="0.04" />
-  <xacro:property name="wheel_radius" value="0.06" />
-  <xacro:macro name="wheel" params="name reflect_x reflect_y reflect_r reflect_axis">
-    <link name="${name}_wheel">
-      <visual>
-        <geometry>
-          <cylinder length="${wheel_height}" radius="${wheel_radius}"/>
-        </geometry>
-        <material name="blue"/>
-      </visual>
-      <collision>
-        <geometry>
-          <cylinder length="${wheel_height}" radius="${wheel_radius}"/>
-        </geometry>
-      </collision>
-      <inertial>
-        <mass value="0.5"/>
-        <inertia ixx="0.001" ixy="0.0" ixz="0.0" iyy="0.001" iyz="0.0" izz="0.001"/>
-      </inertial>
+<robot xmlns:xacro="http://www.ros.org/wiki/xacro" >
+    <xacro:include filename="inertial_macros.xacro"/>
+    <material name="white"><color rgba="1 1 1 1" /></material>
+    <material name="orange"><color rgba="1 0.3 0.1 1"/></material>
+    <material name="blue"><color rgba="0.2 0.2 1 1"/></material>
+    <material name="black"><color rgba="0 0 0 1"/></material>
+    <material name="red"><color rgba="1 0 0 1"/></material>
+    <link name="base_link"></link>
+    <joint name="chassis_joint" type="fixed">
+        <parent link="base_link"/>
+        <child link="chassis"/>
+        <origin xyz="-0.1 0 0"/>
+    </joint>
+    <link name="chassis">
+        <visual>
+            <origin xyz="0.15 0 0.075"/>
+            <geometry>
+                <box size="0.3 0.3 0.15"/>
+            </geometry>
+            <material name="white"/>
+        </visual>
+        <collision>
+            <origin xyz="0.15 0 0.075"/>
+            <geometry>
+                <box size="0.3 0.3 0.15"/>
+            </geometry>
+        </collision>
+        <xacro:inertial_box mass="0.5" x="0.3" y="0.3" z="0.15">
+            <origin xyz="0.15 0 0.075" rpy="0 0 0"/>
+        </xacro:inertial_box>
     </link>
-    <joint name="${name}_wheel_joint" type="continuous">
-      <parent link="chassis"/>
-      <child link="${name}_wheel"/>
-      <origin xyz="${reflect_x*height/2} ${reflect_y*(width/2+0.025)} -0.05" rpy="${reflect_r*1.5707} 0 0"/>
-      <axis xyz="0 0 ${reflect_axis}"/>
-    </joint>
-    <gazebo reference="${name}_wheel">
-      <material>Gazebo/Blue</material>
+    <gazebo reference="chassis">
+        <material>Gazebo/White</material>
     </gazebo>
-  </xacro:macro>
-  <xacro:wheel name="front_right" reflect_x="1" reflect_y="-1" reflect_r="1" reflect_axis="-1"/>
-  <xacro:wheel name="front_left" reflect_x="1" reflect_y="1" reflect_r="-1" reflect_axis="1"/>
-  <xacro:wheel name="rear_right" reflect_x="-1" reflect_y="-1" reflect_r="1" reflect_axis="-1"/>
-  <xacro:wheel name="rear_left" reflect_x="-1" reflect_y="1" reflect_r="-1" reflect_axis="1"/>
-  <material name="green">
-    <color rgba="0 0.8 0 1"/>
-  </material>
-  <link name="head">
-    <visual>
-      <geometry>
-        <box size="0.04 0.04 0.04"/>
-      </geometry>
-      <material name="green"/>
-    </visual>
-  </link>
-  <joint name="head_joint" type="fixed">
-    <parent link="chassis"/>
-    <child link="head"/>
-    <origin xyz="0.1 0 0.07" rpy="0 0 0"/>
-  </joint>
-  <gazebo reference="head">
-    <material>Gazebo/Green</material>
-  </gazebo>
-  <gazebo>
-    <plugin name="skid_steer_drive_controller" filename="libgazebo_ros_skid_steer_drive.so">
-      <updateRate>100.0</updateRate>
-      <robotNamespace>/</robotNamespace>
-      <leftFrontJoint>front_left_wheel_joint</leftFrontJoint>
-      <rightFrontJoint>front_right_wheel_joint</rightFrontJoint>
-      <leftRearJoint>rear_left_wheel_joint</leftRearJoint>
-      <rightRearJoint>rear_right_wheel_joint</rightRearJoint>
-      <wheelSeparation>0.4</wheelSeparation>
-      <wheelDiameter>0.12</wheelDiameter>
-      <torque>20</torque>
-      <commandTopic>cmd_vel</commandTopic>
-      <odometryTopic>odom</odometryTopic>
-      <odometryFrame>odom</odometryFrame>
-      <robotBaseFrame>base_link</robotBaseFrame>
-      <broadcastTF>true</broadcastTF>
-    </plugin>
-  </gazebo>
+    <xacro:macro name="wheel" params="prefix x_reflect y_reflect">
+        <link name="${prefix}_wheel">
+            <visual>
+                <geometry>
+                    <cylinder radius="0.05" length="0.04"/>
+                </geometry>
+                <material name="blue"/>
+            </visual>
+            <collision>
+                <geometry>
+                    <cylinder radius="0.05" length="0.04"/>
+                </geometry>
+            </collision>
+            <xacro:inertial_cylinder mass="0.1" length="0.04" radius="0.05">
+                <origin xyz="0 0 0" rpy="0 0 0"/>
+            </xacro:inertial_cylinder>
+        </link>
+        <joint name="${prefix}_wheel_joint" type="continuous">
+            <parent link="base_link"/>
+            <child link="${prefix}_wheel"/>
+            <origin xyz="${x_reflect*0.1} ${y_reflect*0.175} 0" rpy="-${pi/2} 0 0"/>
+            <axis xyz="0 0 1"/>
+        </joint>
+        <gazebo reference="${prefix}_wheel">
+            <material>Gazebo/Blue</material>
+            <mu1>0.2</mu1>
+            <mu2>0.4</mu2>
+        </gazebo>
+    </xacro:macro>
+    <xacro:wheel prefix="front_left" x_reflect="1" y_reflect="1" />
+    <xacro:wheel prefix="front_right" x_reflect="1" y_reflect="-1" />
+    <xacro:wheel prefix="rear_left" x_reflect="-1" y_reflect="1" />
+    <xacro:wheel prefix="rear_right" x_reflect="-1" y_reflect="-1" />
 </robot>

Commit message: update file

File: urdf/gazebo_control.xacro (robot description, xacro)
@@ -2,14 +2,19 @@
 <robot xmlns:xacro="http://www.ros.org/wiki/xacro">
   <gazebo>
-    <plugin name="mecanum_controller" filename="libgazebo_ros_planar_move.so">
-      <commandTopic>cmd_vel</commandTopic>
+    <plugin name="skid_steer_drive_controller" filename="libgazebo_ros_skid_steer_drive.so">
+      <updateRate>100.0</updateRate>
+      <robotNamespace>/</robotNamespace>
+      <leftFrontJoint>front_left_wheel_joint</leftFrontJoint>
+      <rightFrontJoint>front_right_wheel_joint</rightFrontJoint>
+      <leftRearJoint>rear_left_wheel_joint</leftRearJoint>
+      <rightRearJoint>rear_right_wheel_joint</rightRearJoint>
+      <wheelSeparation>0.4</wheelSeparation> <wheelDiameter>0.2</wheelDiameter>   <robotBaseFrame>base_link</robotBaseFrame>
+      <torque>20</torque>
+      <topicName>cmd_vel</topicName>
       <odometryTopic>odom</odometryTopic>
       <odometryFrame>odom</odometryFrame>
-      <odometryRate>20.0</odometryRate>
-      <robotBaseFrame>base_link</robotBaseFrame>
-      <accelX>10.0</accelX>
-      <accelY>10.0</accelY>
-      <accelTheta>20.0</accelTheta>
-    </plugin> <plugin name="joint_state_publisher" filename="libgazebo_ros_joint_state_publisher.so">
+      <broadcastTF>true</broadcastTF>
+    </plugin>
+    <plugin name="joint_state_publisher" filename="libgazebo_ros_joint_state_publisher.so">
       <robotNamespace>/</robotNamespace>
       <jointName>front_left_wheel_joint, front_right_wheel_joint, rear_left_wheel_joint, rear_right_wheel_joint</jointName>

File: urdf/robot_core.xacro (robot description, xacro)
@@ -8,6 +8,6 @@
     <xacro:property name="chassis_mass"   value="2.0"/>
     <!-- Bánh xe-->
-    <xacro:property name="wheel_radius" value="0.05"/>
-    <xacro:property name="wheel_width"  value="0.04"/>
+    <xacro:property name="wheel_radius" value="0.03"/>
+    <xacro:property name="wheel_width"  value="0.026"/>
     <xacro:property name="wheel_mass"   value="0.2"/>
     <xacro:property name="wheel_track" value="0.44"/>
